File: pcb/main/main.kicad_pcb (KiCad board)
At the start: 2 copper layers, 26 x 13.6 mm, 36 parts, among them J1 USBMCS1B5W, J2 Screw_Terminal_01x03/3,5, J4 Conn_01x04_Male, J5 Conn_01x02_Female, U1 MCP1700-3302E_SOT23, U2 MCP2542FDxMF, U3 USBLC6-2SC6, U4 STM32G431CBUx

Commit message: Text update
Parts:
- removed TP9: TestPoint, Measurement_Points:Measurement_Point_Round-SMD-Pad_Small
Routing:
- net GND: track 88.6 -> 87.6 mm
- net Net-(J5-Pad2): track 6.85 -> 7.84 mm
Other:
- board text added: "D+"
- board text added: "D-"
- board text added: "VCC"
Changed lines of the file:
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@@
   (general
     (thickness 1.6)
-    (drawings 13)
-    (tracks 318)
+    (drawings 17)
+    (tracks 320)
     (zones 0)
-    (modules 36)
+    (modules 35)
     (nets 58)
   )
@@
     (add_net VB_N)
   )
+  (module Pin_Header_Straight_1x02_Pitch2.54mm (layer B.Cu)
+    (at 26.1874 25.6794 90)
+    (descr "Through hole straight pin header, 1x02, 2.54mm pitch, single row")
+    (tags "Through hole pin header THT 1x02 2.54mm single row")
+    (fp_text reference J5 (at 0.762 1.5748 90) (layer B.SilkS)
+      (effects (font (size 0.5 0.5) (thickness 0.1)) (justify mirror))
+    )
+    (fp_text value Conn_01x02_Female (at 0 -4.87 90) (layer B.Fab)
+      (effects (font (size 1 1) (thickness 0.15)) (justify mirror))
+    )
+    (fp_text user %R (at 0 -1.27) (layer B.Fab)
+      (effects (font (size 1 1) (thickness 0.15)) (justify mirror))
+    )
+    (fp_line (start 1.8 1.8) (end -1.8 1.8) (layer B.CrtYd) (width 0.05))
+    (fp_line (start 1.8 -4.35) (end 1.8 1.8) (layer B.CrtYd) (width 0.05))
+    (fp_line (start -1.8 -4.35) (end 1.8 -4.35) (layer B.CrtYd) (width 0.05))
+    (fp_line (start -1.8 1.8) (end -1.8 -4.35) (layer B.CrtYd) (width 0.05))
+    (fp_line (start -1.33 1.33) (end 0 1.33) (layer B.SilkS) (width 0.12))
+    (fp_line (start -1.33 0) (end -1.33 1.33) (layer B.SilkS) (width 0.12))
+    (fp_line (start -1.33 -1.27) (end 1.33 -1.27) (layer B.SilkS) (width 0.12))
+    (fp_line (start 1.33 -1.27) (end 1.33 -3.87) (layer B.SilkS) (width 0.12))
+    (fp_line (start -1.33 -1.27) (end -1.33 -3.87) (layer B.SilkS) (width 0.12))
+    (fp_line (start -1.33 -3.87) (end 1.33 -3.87) (layer B.SilkS) (width 0.12))
+    (fp_line (start -1.27 0.635) (end -0.635 1.27) (layer B.Fab) (width 0.1))
+    (fp_line (start -1.27 -3.81) (end -1.27 0.635) (layer B.Fab) (width 0.1))
+    (fp_line (start 1.27 -3.81) (end -1.27 -3.81) (layer B.Fab) (width 0.1))
+    (fp_line (start 1.27 1.27) (end 1.27 -3.81) (layer B.Fab) (width 0.1))
+    (fp_line (start -0.635 1.27) (end 1.27 1.27) (layer B.Fab) (width 0.1))
+    (pad 2 thru_hole oval (at 0 -2.54 90) (size 1.7 1.7) (drill 1) (layers *.Cu *.Mask)
+      (net 15 "Net-(J5-Pad2)"))
+    (pad 1 thru_hole rect (at 0 0 90) (size 1.7 1.7) (drill 1) (layers *.Cu *.Mask)
+      (net 55 /CANH))
+    (pad 2 smd rect (at 0.1 1.6) (size 1 2) (layers F.Cu F.Paste F.Mask)
+      (net 15 "Net-(J5-Pad2)"))
+    (model ${KISYS3DMOD}/Pin_Headers.3dshapes/Pin_Header_Straight_1x02_Pitch2.54mm.wrl
+      (at (xyz 0 0 0))
+      (scale (xyz 1 1 1))
+      (rotate (xyz 0 0 0))
+    )
+  )
   (module TerminalBlocks_Phoenix:TerminalBlock_Phoenix_PT-3.5mm_3pol (layer B.Cu)
     (at 25.527 29.5402 270)
@@
     )
   )
-  (module Pin_Header_Straight_1x02_Pitch2.54mm (layer B.Cu)
-    (at 26.1874 25.6794 90)
-    (descr "Through hole straight pin header, 1x02, 2.54mm pitch, single row")
-    (tags "Through hole pin header THT 1x02 2.54mm single row")
-    (fp_text reference J5 (at 0.762 1.5748 90) (layer B.SilkS)
-      (effects (font (size 0.5 0.5) (thickness 0.1)) (justify mirror))
-    )
-    (fp_text value Conn_01x02_Female (at 0 -4.87 90) (layer B.Fab)
-      (effects (font (size 1 1) (thickness 0.15)) (justify mirror))
-    )
-    (fp_text user %R (at 0 -1.27 180) (layer B.Fab)
-      (effects (font (size 1 1) (thickness 0.15)) (justify mirror))
-    )
-    (fp_line (start 1.8 1.8) (end -1.8 1.8) (layer B.CrtYd) (width 0.05))
-    (fp_line (start 1.8 -4.35) (end 1.8 1.8) (layer B.CrtYd) (width 0.05))
-    (fp_line (start -1.8 -4.35) (end 1.8 -4.35) (layer B.CrtYd) (width 0.05))
-    (fp_line (start -1.8 1.8) (end -1.8 -4.35) (layer B.CrtYd) (width 0.05))
-    (fp_line (start -1.33 1.33) (end 0 1.33) (layer B.SilkS) (width 0.12))
-    (fp_line (start -1.33 0) (end -1.33 1.33) (layer B.SilkS) (width 0.12))
-    (fp_line (start -1.33 -1.27) (end 1.33 -1.27) (layer B.SilkS) (width 0.12))
-    (fp_line (start 1.33 -1.27) (end 1.33 -3.87) (layer B.SilkS) (width 0.12))
-    (fp_line (start -1.33 -1.27) (end -1.33 -3.87) (layer B.SilkS) (width 0.12))
-    (fp_line (start -1.33 -3.87) (end 1.33 -3.87) (layer B.SilkS) (width 0.12))
-    (fp_line (start -1.27 0.635) (end -0.635 1.27) (layer B.Fab) (width 0.1))
-    (fp_line (start -1.27 -3.81) (end -1.27 0.635) (layer B.Fab) (width 0.1))
-    (fp_line (start 1.27 -3.81) (end -1.27 -3.81) (layer B.Fab) (width 0.1))
-    (fp_line (start 1.27 1.27) (end 1.27 -3.81) (layer B.Fab) (width 0.1))
-    (fp_line (start -0.635 1.27) (end 1.27 1.27) (layer B.Fab) (width 0.1))
-    (pad 2 thru_hole oval (at 0 -2.54 90) (size 1.7 1.7) (drill 1) (layers *.Cu *.Mask)
-      (net 15 "Net-(J5-Pad2)"))
-    (pad 1 thru_hole rect (at 0 0 90) (size 1.7 1.7) (drill 1) (layers *.Cu *.Mask)
-      (net 55 /CANH))
-    (model ${KISYS3DMOD}/Pin_Headers.3dshapes/Pin_Header_Straight_1x02_Pitch2.54mm.wrl
-      (at (xyz 0 0 0))
-      (scale (xyz 1 1 1))
-      (rotate (xyz 0 0 0))
-    )
-  )
   (module Measurement_Points:Measurement_Point_Round-SMD-Pad_Small (layer F.Cu)
     (at 36.195 28.067)
@@
     (attr virtual)
     (fp_text reference TP5 (at 0 -1.397) (layer F.SilkS)
-      (effects (font (size 0.3 0.3) (thickness 0.075)))
+      (effects (font (size 0.5 0.5) (thickness 0.125)))
     )
     (fp_text value TestPoint (at 0 2) (layer F.Fab)
@@
       (net 3 +3V3))
   )
-  (module Measurement_Points:Measurement_Point_Round-SMD-Pad_Small (layer F.Cu)
-    (at 42.418 28.956)
-    (descr "Mesurement Point, Round, SMD Pad, DM 1.5mm,")
-    (tags "Mesurement Point Round SMD Pad 1.5mm")
-    (attr virtual)
-    (fp_text reference TP9 (at -1.27 -0.381 90) (layer F.SilkS)
-      (effects (font (size 0.4 0.4) (thickness 0.1)))
-    )
-    (fp_text value TestPoint (at 0 2) (layer F.Fab)
-      (effects (font (size 1 1) (thickness 0.15)))
-    )
-    (fp_circle (center 0 0) (end 1 0) (layer F.CrtYd) (width 0.05))
-    (pad 1 smd circle (at 0 0) (size 1.5 1.5) (layers F.Cu F.Mask)
-      (net 1 GND))
+  (gr_text GND (at 46.99 34.417) (layer F.SilkS)
+    (effects (font (size 0.3 0.3) (thickness 0.075)))
+  )
+  (gr_text D+ (at 45.72 34.417) (layer F.SilkS)
+    (effects (font (size 0.3 0.3) (thickness 0.075)))
+  )
+  (gr_text D- (at 45.593 31.496) (layer F.SilkS)
+    (effects (font (size 0.3 0.3) (thickness 0.075)))
+  )
+  (gr_text VCC (at 46.863 31.496) (layer F.SilkS)
+    (effects (font (size 0.3 0.3) (thickness 0.075)))
   )
   (gr_text CANH (at 27.432 33.02 90) (layer F.SilkS)
@@
   )
   (gr_text GND (at 23.241 29.591 90) (layer F.SilkS)
-    (effects (font (size 1 1) (thickness 0.2)))
+    (effects (font (size 0.7 0.7) (thickness 0.175)))
   )
   (gr_text CANL (at 23.368 36.322 90) (layer F.SilkS)
-    (effects (font (size 1 1) (thickness 0.2)))
+    (effects (font (size 0.7 0.7) (thickness 0.175)))
   )
   (gr_text ucandevices.github.io (at 43.942 37.465) (layer B.SilkS)
@@
   (via (at 41.401099 28.956901) (size 0.8) (drill 0.4) (layers F.Cu B.Cu) (net 1))
   (segment (start 41.401099 28.956901) (end 41.986398 29.5422) (width 0.25) (layer B.Cu) (net 1))
-  (segment (start 42.418 28.956) (end 41.402 28.956) (width 0.25) (layer F.Cu) (net 1))
   (segment (start 39.8881 28.7264) (end 39.497 28.3353) (width 0.25) (layer B.Cu) (net 2))
   (segment (start 39.497 28.3353) (end 39.497 28.2723) (width 0.25) (layer B.Cu) (net 2))
@@
   (segment (start 31.1524 27.939542) (end 30.439631 28.652311) (width 0.25) (layer F.Cu) (net 3))
   (segment (start 31.1524 27.4828) (end 31.1524 27.939542) (width 0.25) (layer F.Cu) (net 3))
-  (segment (start 28.5863 37.3493) (end 35.8956 37.3493) (width 0.25) (layer F.Cu) (net 3))
+  (segment (start 41.8617 36.195) (end 42.926 36.195) (width 0.25) (layer F.Cu) (net 3))
+  (segment (start 41.4673 36.5894) (end 41.8617 36.195) (width 0.25) (layer F.Cu) (net 3))
+  (segment (start 35.6529 37.592) (end 35.8956 37.3493) (width 0.25) (layer F.Cu) (net 3))
+  (segment (start 28.829 37.592) (end 35.6529 37.592) (width 0.25) (layer F.Cu) (net 3))
   (segment (start 30.6456 30.524) (end 29.368597 29.246997) (width 0.25) (layer F.Cu) (net 3))
   (segment (start 31.2456 30.524) (end 30.6456 30.524) (width 0.25) (layer F.Cu) (net 3))
@@
   (segment (start 27.718998 29.246997) (end 27.34199 29.624005) (width 0.25) (layer F.Cu) (net 3))
   (segment (start 27.34199 29.624005) (end 27.34199 36.10499) (width 0.25) (layer F.Cu) (net 3))
-  (segment (start 27.34199 36.10499) (end 28.5863 37.3493) (width 0.25) (layer F.Cu) (net 3))
-  (segment (start 41.8617 36.195) (end 42.926 36.195) (width 0.25) (layer F.Cu) (net 3))
-  (segment (start 41.4673 36.5894) (end 41.8617 36.195) (width 0.25) (layer F.Cu) (net 3))
+  (segment (start 27.34199 36.10499) (end 28.829 37.592) (width 0.25) (layer F.Cu) (net 3))
   (segment (start 34.3956 29.4262) (end 35.065801 28.755999) (width 0.25) (layer F.Cu) (net 4))
   (segment (start 34.278 26.5826) (end 34.278 25.8826) (width 0.25) (layer F.Cu) (net 4))
@@
   (segment (start 23.3172 27.1849) (end 23.3172 31.9398) (width 0.25) (layer F.Cu) (net 15))
   (segment (start 23.3172 31.9398) (end 23.3172 32.397) (width 0.25) (layer F.Cu) (net 15))
+  (segment (start 24.4874 25.6794) (end 24.5874 25.5794) (width 0.25) (layer F.Cu) (net 15))
+  (segment (start 23.6474 25.6794) (end 24.4874 25.6794) (width 0.25) (layer F.Cu) (net 15))
   (segment (start 45.962 28.702) (end 45.835 28.575) (width 0.25) (layer F.Cu) (net 16))
   (via (at 46.9265 28.321) (size 0.8) (drill 0.4) (layers F.Cu B.Cu) (net 16))
