File: pcb/main/main.sch (KiCad schematic (older format))
At the start: 36 parts, among them J1 USBMCS1B5W, J2 Screw_Terminal_01x03/3,5, J4 Conn_01x04_Male, J5 Conn_01x02_Female, U1 MCP1700-3302E_SOT23, U2 MCP2542FDxMF, U3 USBLC6-2SC6, U4 STM32G431CBUx

Commit message: Text update
Parts:
- removed TP9: TestPoint, Measurement_Points:Measurement_Point_Round-SMD-Pad_Small, symbol Connector:TestPoint
Changed lines of the file:
@@
-$EndComp
-$Comp
-L Connector:TestPoint TP9
-U 1 1 5ECD5181
-P 3650 4050
-F 0 "TP9" V 3604 4238 50  0000 L CNN
-F 1 "TestPoint" V 3695 4238 50  0001 L CNN
-F 2 "Measurement_Points:Measurement_Point_Round-SMD-Pad_Small" H 3850 4050 50  0001 C CNN
-F 3 "~" H 3850 4050 50  0001 C CNN
-	1    3650 4050
-	1    0    0    -1
-$EndComp
-$Comp
-L power:GND #PWR0110
-U 1 1 5ECD530A
-P 3650 4050
-F 0 "#PWR0110" H 3650 3800 50  0001 C CNN
-F 1 "GND" H 3655 3877 50  0000 C CNN
-F 2 "" H 3650 4050 50  0001 C CNN
-F 3 "" H 3650 4050 50  0001 C CNN
-	1    3650 4050
-	-1   0    0    -1
 $EndComp
 $Comp
